File: hardware/allie-reader/allie-reader.kicad_sch (KiCad schematic)
At the start: 17 parts, among them J1 8P8C Socket, J2 Reader, U1 MAX488E, U2 LD1117S50TR, U3 CH32V003JxMx

Commit message: add: pcb for allie
Parts:
- removed C4: 0.1u 16V, symbol Device:C_Small
- removed U3: CH32V003JxMx, Package_SO:JEITA_SOIC-8_3.9x4.9mm_P1.27mm, symbol MCU_WCH_RiscV:CH32V003JxMx
- added BZ1: Buzzer, Used_Symbols:Buzzer_17mm, symbol Device:Buzzer
- added C5, C6, C7: 0.1u 16V, Capacitor_SMD:C_0805_2012Metric, symbol Device:C_Small
- added D6: SM712, Package_TO_SOT_SMD:SOT-23, symbol Diode:SM712_SOT23
- added J3: LED, Connector_JST:JST_XH_B3B-XH-A_1x03_P2.50mm_Vertical, symbol Connector:Conn_01x03_Socket
- added JMP1, JMP2, JMP3, JMP4, JMP5, JMP6: 0, Resistor_SMD:R_1206_3216Metric, symbol Device:R
- added Q1: AO3401A, Package_TO_SOT_SMD:SOT-23, symbol Transistor_FET:AO3401A
- added R3: 5.1k, Resistor_SMD:R_0805_2012Metric, symbol Device:R
- added R4, R5: 240, Resistor_SMD:R_0805_2012Metric, symbol Device:R
- added TP1: SWIO, TestPoint:TestPoint_Pad_D2.0mm, symbol Connector:TestPoint
- added TP2: GND, TestPoint:TestPoint_Pad_D2.0mm, symbol Connector:TestPoint
- added U4: SN75176AD, Package_SO:SOIC-8_3.9x4.9mm_P1.27mm, symbol Interface_UART:SN75176AD
- added U5: CH32V003AxMx, Package_SO:SOP-16_3.9x9.9mm_P1.27mm, symbol MCU_WCH_CH32V0:CH32V003AxMx
- C1, C2, C3: footprint (none) -> Capacitor_SMD:C_0805_2012Metric
- D5: footprint (none) -> LED_SMD:LED_0805_2012Metric
- J1: footprint (none) -> Connector_JST:JST_XH_B8B-XH-A_1x08_P2.50mm_Vertical
Connections:
- net RDR_GND is gone; now on net GND: J2.1 (Pin_1)
- net +5V: now also C5.1, C6.1, J3.3 (Pin_3), JMP2.1, JMP2.2, JMP5.1, JMP5.2, Q1.3 (D), R3.1, U4.8 (VCC), U5.15 (VDD)
- net GND: now also BZ1.2 (-), C5.2, C6.2, C7.1, D6.3 (common), J3.1 (Pin_1), JMP3.1, JMP3.2, JMP4.1, JMP4.2, TP2.1, U4.5 (GND), U5.14 (VSS)
- net LED_DATA: now also J3.2 (Pin_2), JMP6.1, JMP6.2, U5.16 (PC0)
- net RDR_PWR_CTRL: now also R4.1, U5.1 (PC1)
- net RDR_VCC: now also Q1.2 (S)
- net RRX_A: now also J1.4 (Pin_4); no longer J1.7 (Pin_7)
- net RRX_B: now also J1.5 (Pin_5); no longer J1.8 (Pin_8)
- net RTX_A: now also D2.2 (A2), J1.8 (Pin_8); no longer D2.1 (A1), J1.5 (Pin_5)
- net RTX_B: now also D2.1 (A1), J1.7 (Pin_7); no longer D2.2 (A2), J1.4 (Pin_4)
- net SBU_A: now also J1.2 (Pin_2), D6.2 (A2), U4.6 (A); no longer J1.1 (Pin_1)
- net SBU_B: now also J1.1 (Pin_1), D6.1 (A1), U4.7 (B); no longer J1.2 (Pin_2)
- net SBU_RX: now also U4.1 (R), U5.10 (PD6)
- net SBU_TX: now also U4.4 (D), U5.9 (PD5)
- net SBU_TXEN: now also JMP1.1, JMP1.2, U4.2 (~{RE}), U4.3 (DE), U5.8 (PD4)
- net SPKR: now also R5.2, U5.6 (PC7)
- new net: BZ1.1 (+), R5.1
- new net: Q1.1 (G), R3.2, R4.2
- new net: C7.2, U5.11 (PD7)
- new net SWIO: TP1.1, U5.7 (PD1)
- no-connect marks 0 -> 6
Other:
- note added: "Reader power"
- note added: "SBU MCU"
- note added: "SBU RS485"
- note added: "SBU buzzer"
- moved on the sheet: J1, J2
